File: Hardware/KiCad/Aquaponic Controller/Aquaponic Controller.sch (KiCad schematic (older format))
At the start: 6 parts

Commit message: Version 1.0
The hardware is working The software still needs work.
Parts:
- added C?: 10K, symbol Device:CP1
- added J?: Conn_01x03, symbol Connector_Generic:Conn_01x03
- added J?: Conn_01x04, symbol Connector_Generic:Conn_01x04
- added J? (x3): Conn_01x02, symbol Connector_Generic:Conn_01x02
- added R? (x2): 10K, symbol Aquaponic-Controller-rescue:R-resistors
- R? (x2): symbol resistors:R -> Aquaponic-Controller-rescue:R-resistors
- R?: value R -> 10K; symbol resistors:R -> Aquaponic-Controller-rescue:R-resistors
- U?: symbol modules:MP1584Module -> Aquaponic-Controller-rescue:MP1584Module-modules
Connections:
- net labels added: Echo, Trig, Vin
- net labels removed: -VDC
- wire segments 35 -> 73
Other:
- note added: "Current sensor"
- note added: "LM35\nTemperature sensor"
- note added: "Ping sensor"
- note added: "Power in\n7 - 12V"
- note added: "relay"
- moved on the sheet: R?
